Commit message: added inertial properties to base model

File: description/urdf/left_leg.xacro (robot description, xacro)
@@ -23,4 +23,10 @@
             </geometry>
         </collision>
+        <inertial>
+            <origin xyz="0.00119 0 -0.03859" rpy="0 0 0"/>
+            <mass value="0.04038"/>
+            <inertia ixx="0.000024549"  ixy="0"  ixz="0.000000183"
+            iyy="0.000018945" iyz="0" izz="0.000007508"/>
+        </inertial>
     </link>
     <!-- TIBIA LINK -->
@@ -46,4 +52,10 @@
             </geometry>
         </collision>
+        <inertial>
+            <origin xyz="0.00447 0 -0.02276" rpy="0 0 0"/>
+            <mass value="0.01338"/>
+            <inertia ixx="0.000008839"  ixy="0"  ixz="0.000001782"
+            iyy="0.000009491" iyz="0" izz="0.000001336"/>
+        </inertial>
     </link>
     <!-- FOOT LINK -->
@@ -69,4 +81,10 @@
             </geometry>
         </collision>
+        <inertial>
+            <origin xyz="-0.00689 0 -0.03048" rpy="0 0 0"/>
+            <mass value="0.04904"/>
+            <inertia ixx="0.000023179"  ixy="0"  ixz="-0.000001838"
+            iyy="0.000038895" iyz="0" izz="0.000040501"/>
+        </inertial>
     </link>
 </robot>

File: description/urdf/right_leg.xacro (robot description, xacro)
@@ -23,4 +23,10 @@
             </geometry>
         </collision>
+        <inertial>
+            <origin xyz="0.00119 0 -0.03859" rpy="0 0 0"/>
+            <mass value="0.04038"/>
+            <inertia ixx="0.000024549"  ixy="0"  ixz="0.000000183"
+            iyy="0.000018945" iyz="0" izz="0.000007508"/>
+        </inertial>
     </link>
     <!-- TIBIA LINK -->
@@ -46,4 +52,10 @@
             </geometry>
         </collision>
+        <inertial>
+            <origin xyz="0.00447 0 -0.02276" rpy="0 0 0"/>
+            <mass value="0.01338"/>
+            <inertia ixx="0.000008839"  ixy="0"  ixz="0.000001782"
+            iyy="0.000009491" iyz="0" izz="0.000001336"/>
+        </inertial>
     </link>
     <!-- FOOT LINK -->
@@ -69,4 +81,10 @@
             </geometry>
         </collision>
+        <inertial>
+            <origin xyz="-0.00689 0 -0.03048" rpy="0 0 0"/>
+            <mass value="0.04904"/>
+            <inertia ixx="0.000023179"  ixy="0"  ixz="-0.000001838"
+            iyy="0.000038895" iyz="0" izz="0.000040501"/>
+        </inertial>
     </link>
 </robot>

File: description/urdf/robot_core.xacro (robot description, xacro)
@@ -23,4 +23,10 @@
             </geometry>
         </collision>
+        <inertial>
+            <origin xyz="-0.00335 0 0.04408" rpy="0 0 0"/>
+            <mass value="0.710"/>
+            <inertia ixx="0.001020342"  ixy="-0.000029751"  ixz="0.000081459"
+            iyy="0.001357339" iyz="-0.000026283" izz="0.001569161"/>
+        </inertial>
     </link>
     <!-- LEFT HIP LINK -->
@@ -46,4 +52,10 @@
             </geometry>
         </collision>
+        <inertial>
+            <origin xyz="-0.001594 -0.00051 -0.04019" rpy="0 0 0"/>
+            <mass value="0.14121"/>
+            <inertia ixx="0.000068413"  ixy="-0.000000090"  ixz="0.000027110"
+            iyy="0.000093037" iyz="0.000000657" izz="0.000068140"/>
+        </inertial>
     </link>
     <!-- RIGHT HIP LINK -->
@@ -69,4 +81,10 @@
             </geometry>
         </collision>
+        <inertial>
+            <origin xyz="-0.001594 0.00051 -0.04019" rpy="0 0 0"/>
+            <mass value="0.14121"/>
+            <inertia ixx="0.000068413"  ixy="0.000000090"  ixz="0.000027110"
+            iyy="0.000093037" iyz="-0.000000657" izz="0.000068140"/>
+        </inertial>
     </link>
 </robot>
